File: hardware/Amp386/Amp386.sch (KiCad schematic (older format))
At the start: 34 parts

Commit message: More schematic
Parts:
- added J?: AudioJack2_Ground_Switch, symbol Connector:AudioJack2_Ground_Switch
- added J?: AudioJack2_Switch, symbol Connector:AudioJack2_Switch
- added LS?: Speaker, symbol Device:Speaker
- added LS?: Earphone, symbol Device:Earphone
- C?: value C_Small -> .001
- C? (x2): value CP_Small -> 10
- C?: value CP_Small -> 330
- R?: value R_Small_US -> 10
Connections:
- net GND: now also C?.2, C?.2, C?.2, RV?.3, U?.2 (-), U?.4 (GND)
- net at U?.1 (GAIN): now also C?.1
- net at U?.3 (+): now also C?.1, RV?.2
- net at U?.5: now also C?.1, C?.1
- net at U?.6 (V+): now also C?.1, R?.2
- net at U?.7 (BYPASS): now also C?.1
- net at U?.8 (GAIN): now also C?.2
- net at C?.2: now also RV?.1
Other:
- moved on the sheet: C?, R?, RV?
